Commit message: Added joystick control and gazebo sim

File: description/robot_core.xacro (robot description, xacro)
@@ -39,4 +39,7 @@
         </xacro:inertial_box>
     </link>
+    <gazebo reference="chassis">
+        <material>Gazebo/White</material>
+    </gazebo>
     <!-- Left wheel link -->
     <joint name="left_wheel_joint" type="continuous">
@@ -62,4 +65,7 @@
         </xacro:inertial_cylinder>
     </link>
+    <gazebo reference="left_wheel">
+        <material>Gazebo/Blue</material>
+    </gazebo>
     <!-- Right wheel link -->
     <joint name="right_wheel_joint" type="continuous">
@@ -85,4 +91,7 @@
         </xacro:inertial_cylinder>
     </link>
+    <gazebo reference="right_wheel">
+        <material>Gazebo/Blue</material>
+    </gazebo>
     <!-- Castor wheel link -->
     <joint name="castor_wheel_joint" type="fixed">
@@ -107,3 +116,8 @@
         </xacro:inertial_sphere>
     </link>
+    <gazebo reference="castor_wheel">
+        <material>Gazebo/Black</material>
+        <mu1 value="0.001" />
+        <mu2 value="0.001" />
+    </gazebo>
 </robot>

Commit message: Lidar capability added

File: description/robot_core.xacro (robot description, xacro)
@@ -6,11 +6,14 @@
     </material>
     <material name="orange">
-        <color rgba="1 0.3 0.1 0.0"/>
+        <color rgba="1 0.3 0.1 1.0"/>
     </material>
     <material name="blue">
-        <color rgba="0.2 0.2 1 0.0"/>
+        <color rgba="0.2 0.2 1 1.0"/>
     </material>
     <material name="black">
-        <color rgba="0.0 0.0 0.0 0.0"/>
+        <color rgba="0.0 0.0 0.0 1.0"/>
+    </material>
+    <material name="red">
+        <color rgba="1.0 0.0 0.0 1.0"/>
     </material>
     <link name="base_link">
